File: bbq10_keyboard.kicad_pcb (KiCad board)
At the start: 2 copper layers, 68 x 45 mm, 20 parts, among them J1 PMOD, Q1 BSS138, U1 BBQ10KBD, U2 ATSAMD20E16A

Commit message: USB BBQ10 keyboard rev 0.5
Parts:
- removed G***: LOGO, Symbols_Extra:SolderParty-Logo_14.6x13.5mm_SilkScreen
- removed J1: PMOD, Connector_PinHeader_2.54mm_Extra:PMODPinHeader_1x06_P2.54mm_Horizontal
- added J2: USB_B_Micro, library:USB_Micro-B_Molex_47346-0001, F.Cu at (148.1, 79.8)
- added J3: Groveconn4, Connector_JST:JST_SH_BM04B-SRSS-TB_1x04-1MP_P1.00mm_Vertical, F.Cu at (159.8, 79.5)
- added J4: Conn_ARM_JTAG_SWD_10, Connector_PinHeader_1.27mm:PinHeader_2x05_P1.27mm_Vertical_SMD, F.Cu at (135.4, 81.0)
- added R6: 10K, Resistor_SMD:R_0603_1608Metric, B.Cu at (145.1, 83.6)
- added TP6: UART_TX, TestPoint:TestPoint_Pad_D1.0mm, B.Cu at (156.0, 111.8)
- added TP7: UART_TX, TestPoint:TestPoint_Pad_D1.0mm, B.Cu at (162.6, 90.7)
- added TP8: UART_TX, TestPoint:TestPoint_Pad_D1.0mm, B.Cu at (162.6, 93.0)
- added TP9: UART_TX, TestPoint:TestPoint_Pad_D1.0mm, B.Cu at (162.6, 95.2)
- added U3: AP2112K-3.3, Package_TO_SOT_SMD:SOT-23-5, B.Cu at (145.0, 87.9)
- U2: value ATSAMD20E16A -> ATSAMD20E17A; footprint Package_DFN_QFN:QFN-32-1EP_5x5mm_P0.5mm_EP3.45x3.45mm -> Package_QFP:TQFP-32_7x7mm_P0.8mm
- moved R3 5.62 mm to (152.7, 105.7)
- moved R2 5.59 mm to (147.3, 105.7)
- moved C3 5.59 mm to (150.9, 105.7)
- moved C1 5.59 mm to (149.1, 105.7)
- moved R5 4.28 mm to (153.7, 86.6)
- moved R4 4.04 mm to (151.9, 86.6)
- moved C2 3.84 mm to (150.1, 86.6)
- moved R1 3.78 mm to (159.0, 86.4)
- moved Q1 3.55 mm to (156.5, 86.6)
- moved TP4 3.52 mm to (144.5, 111.8)
- moved TP1 3.44 mm to (146.8, 111.8)
- moved TP5 3.42 mm to (149.1, 111.8)
- moved TP2 3.41 mm to (151.4, 111.8)
- moved TP3 3.31 mm to (153.7, 111.8)
- moved U2 2.50 mm to (150.9, 97.0)
Connections:
- net +3V3 renamed VCC
- net Net-(R2-Pad1) renamed SWCLK
- net Net-(TP2-Pad1) renamed SWDIO
- U2 pad 15: Net-(U2-Pad15) -> GPIO0
- U2 pad 16: Net-(U2-Pad16) -> GPIO1
- U2 pad 17: Net-(U2-Pad17) -> /UART_TX
- U2 pad 18: Net-(U2-Pad18) -> UART_RX
- U2 pad 19: Net-(U2-Pad19) -> GPIO2
- U2 pad 20: Net-(U2-Pad20) -> /ROW1
- U2 pad 21: /UART_TX -> /COL1
- U2 pad 22: /ROW1 -> /ROW2
- U2 pad 23: /COL1 -> DM
- U2 pad 24: /ROW2 -> DP
Routing:
- net GND: track 6.08 -> 162.8 mm, vias 6 -> 42
- net /~RESET~: track 2.18 -> 38.0 mm, vias 0 -> 5
- net SWCLK: track 13.6 -> 47.2 mm, vias 2 -> 6
- net VCC: track 53.1 -> 85.1 mm, vias 5 -> 8
- net SWDIO: track 15.0 -> 46.7 mm, vias 2 -> 5
- net DP: track 0.00 -> 28.8 mm, vias 0 -> 1
- net DM: track 0.00 -> 26.2 mm, vias 0 -> 1
- net UART_RX: track 0.00 -> 19.8 mm, vias 0 -> 2
- net /INT: track 13.6 -> 0.00 mm
- net GPIO0: track 0.00 -> 11.3 mm, vias 0 -> 2
- net VIN: track 0.00 -> 10.9 mm, vias 0 -> 1
- net GPIO1: track 0.00 -> 10.5 mm, vias 0 -> 2
- net Net-(Q1-Pad3): track 16.7 -> 25.8 mm
- net GPIO2: track 0.00 -> 8.43 mm, vias 0 -> 2
- net /UART_TX: track 14.8 -> 21.6 mm, vias 0 -> 2
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Other:
- outline, holes or cut-outs redrawn
- board text added: "1"
- board text added: "@hanyazou"
- board text added: "BBQ10KBD"
- board text added: "BBQ10KBD USB Rev 0.5 Mar 2020 @hanyazou Original design by @arturo182"
- board text added: "GPIO0"
- board text added: "GPIO1"
- board text added: "GPIO2"
- board text added: "Qwiic I2C"
- board text added: "RX←"
- board text added: "SWCLK"
- board text added: "SWD"
- board text added: "SWDIO"
- board text added: "TX→"
- board text added: "USB"
- board text added: "●"
- board text removed: "@arturo182"
- board text removed: "BBQ10KBD PMOD"
- board text removed: "BBQ10KBD PMOD rev2 Nov 2018 by @arturo182"
- board text removed: "CLK"
- board text removed: "INT"
- board text removed: "IO"
- board text removed: "SCL"
- board text removed: "SDA"
- board text removed: "TX"

Commit message: USB BBQ10 keyboard rev 0.9
Parts:
- added D1: USR_LED0, LED_SMD:LED_0603_1608Metric_Pad1.05x0.95mm_HandSolder, F.Cu at (167.1, 83.3)
- added D2: USR_LED1, LED_SMD:LED_0603_1608Metric_Pad1.05x0.95mm_HandSolder, F.Cu at (172.3, 83.3)
- added D3: PWR_LED, LED_SMD:LED_0603_1608Metric_Pad1.05x0.95mm_HandSolder, F.Cu at (178.1, 83.3)
- added J5: SWD, library:Conn4 1.0mm pitch, F.Cu at (135.6, 110.9)
- added J6: SWD, Connector_PinHeader_2.54mm:PinHeader_1x04_P2.54mm_Vertical, B.Cu at (129.2, 100.8)
- added J7: GPIO_header, Connector_PinHeader_2.54mm:PinHeader_1x04_P2.54mm_Vertical, B.Cu at (167.0, 100.8)
- added J8: Debug_header, Connector_PinHeader_2.54mm:PinHeader_1x06_P2.54mm_Vertical, B.Cu at (154.4, 108.5)
- added R7: 1K, Resistor_SMD:R_0603_1608Metric_Pad1.05x0.95mm_HandSolder, B.Cu at (166.2, 87.0)
- added R8: 1K, Resistor_SMD:R_0603_1608Metric_Pad1.05x0.95mm_HandSolder, B.Cu at (168.3, 87.0)
- added R9: 220R, Resistor_SMD:R_0603_1608Metric_Pad1.05x0.95mm_HandSolder, B.Cu at (170.2, 87.0)
- added TP10: TP_GPIO3, TestPoint:TestPoint_Pad_D1.0mm, B.Cu at (163.8, 108.5)
- J3: value Groveconn4 -> Qwiic_connector; footprint Connector_JST:JST_SH_BM04B-SRSS-TB_1x04-1MP_P1.00mm_Vertical -> Connector_JST:JST_SH_SM04B-SRSS-TB_1x04-1MP_P1.00mm_Horizontal
- TP3: value UART_TX -> TP_UART_TX
- TP4: value VDD -> TP_VCC
- TP5: value GND -> TP_GND
- TP6: value UART_TX -> TP_UART_RX
- TP7: value UART_TX -> TP_GPIO0
- TP8: value UART_TX -> TP_GPIO1
- TP9: value UART_TX -> TP_GPIO2
- moved TP4 11.5 mm to (154.4, 106.0)
- moved TP2 11.2 mm to (141.7, 106.0)
- moved TP9 10.7 mm to (163.8, 105.9)
- moved TP8 10.5 mm to (163.8, 103.4)
- moved TP7 10.2 mm to (163.8, 100.8)
- moved TP3 7.16 mm to (149.4, 106.0)
- moved TP6 7.01 mm to (151.9, 106.0)
- moved TP1 6.25 mm to (144.3, 106.0)
- moved TP5 6.16 mm to (146.8, 106.0)
- moved R3 4.46 mm to (156.9, 104.3), turned to 180 degrees
- moved C3 2.59 mm to (153.1, 104.3), turned to 0 degrees
- moved REF** 2.35 mm to (124.4, 92.2), turned to 90 degrees
- moved R2 2.33 mm to (145.4, 104.3), turned to 0 degrees
- moved C1 1.34 mm to (149.2, 104.3), turned to 0 degrees
- moved J3 0.74 mm to (159.5, 80.2), turned to 180 degrees
Connections:
- net /UART_TX renamed UART_TX
- net Net-(C3-Pad1) renamed VDDCORE
- U2 pad 27: Net-(U2-Pad27) -> GPIO3
Routing:
- net VCC: track 85.1 -> 132.6 mm, vias 8 -> 9
- net GPIO3: track 0.00 -> 39.9 mm, vias 0 -> 1
- net SWCLK: track 47.2 -> 78.9 mm, vias 6 -> 5
- net SWDIO: track 46.7 -> 75.7 mm
- net GPIO2: track 8.43 -> 34.2 mm, vias 2 -> 3
- net GPIO0: track 11.3 -> 24.7 mm
- net GPIO1: track 10.5 -> 22.5 mm
- net Net-(D3-Pad2): track 0.00 -> 8.16 mm, vias 0 -> 1
- net GND: track 162.8 -> 156.4 mm, vias 42 -> 64
- net Net-(D2-Pad2): track 0.00 -> 4.79 mm, vias 0 -> 1
- net Net-(D1-Pad2): track 0.00 -> 2.81 mm, vias 0 -> 1
- net /SCL: track 18.1 -> 15.7 mm
- net /SDA: track 18.8 -> 16.9 mm
- net UART_TX: track 21.6 -> 23.0 mm
- net DP: track 28.8 -> 28.1 mm
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Other:
- board text added: "BBQ10KBD USB Rev 0.9 April 2020 @hanyazou Original design by @arturo182"
- board text added: "GPIO3"
- board text added: "PWR"
- board text added: "Qwiic"
- board text added: "U0"
- board text added: "U1"
- board text added: "VCC"
- board text added: "VCC RX→ TX← GND SWCLK SWDIO"
- board text removed: "1"
- board text removed: "3V3"
- board text removed: "BBQ10KBD USB Rev 0.5 Mar 2020 @hanyazou Original design by @arturo182"
- board text removed: "Qwiic I2C"
- board text removed: "RX←"
- board text removed: "TX→"
