File: bbq10_keyboard.sch (KiCad schematic (older format))
At the start: 17 parts, among them J1 PMOD, Q1 BSS138, U1 BBQ10KBD, U2 ATSAMD20E16A

Commit message: USB BBQ10 keyboard rev 0.5
Parts:
- removed U2: ATSAMD20E16A, Package_DFN_QFN:QFN-32-1EP_5x5mm_P0.5mm_EP3.45x3.45mm, symbol MCU_Microchip_SAMD:ATSAMD20E16A
- added J2: USB_B_Micro, library:USB_Micro-B_Molex_47346-0001, symbol Connector:USB_B_Micro
- added J3: Groveconn4, Connector_JST:JST_SH_BM04B-SRSS-TB_1x04-1MP_P1.00mm_Vertical, symbol mylib:Groveconn4
- added J4: Conn_ARM_JTAG_SWD_10, Connector_PinHeader_1.27mm:PinHeader_2x05_P1.27mm_Vertical_SMD, symbol Connector:Conn_ARM_JTAG_SWD_10
- added R6: 10K, Resistor_SMD:R_0603_1608Metric, symbol Device:R_Small
- added TP6, TP7, TP8, TP9: UART_TX, TestPoint:TestPoint_Pad_D1.0mm, symbol Connector:TestPoint
- added U2: ATSAMD20E17A, Package_QFP:TQFP-32_7x7mm_P0.8mm, symbol MCU_Microchip_SAMD:ATSAMD20E17A
- added U3: AP2112K-3.3, Package_TO_SOT_SMD:SOT-23-5, symbol Regulator_Linear:AP2112K-3.3
Connections:
- net labels added: DM, DP, GPIO0, GPIO1, GPIO2, SWCLK, SWDIO, UART_RX, VCC, VIN
- wire segments 91 -> 111
- no-connect marks 10 -> 9
Other:
- moved on the sheet: TP1, TP2

Commit message: USB BBQ10 keyboard rev 0.9
Parts:
- removed J3: Groveconn4, Connector_JST:JST_SH_BM04B-SRSS-TB_1x04-1MP_P1.00mm_Vertical, symbol mylib:Groveconn4
- added D1: USR_LED0, LED_SMD:LED_0603_1608Metric_Pad1.05x0.95mm_HandSolder, symbol Device:LED
- added D2: USR_LED1, LED_SMD:LED_0603_1608Metric_Pad1.05x0.95mm_HandSolder, symbol Device:LED
- added D3: PWR_LED, LED_SMD:LED_0603_1608Metric_Pad1.05x0.95mm_HandSolder, symbol Device:LED
- added J3: Qwiic_connector, Connector_JST:JST_SH_SM04B-SRSS-TB_1x04-1MP_P1.00mm_Horizontal, symbol mylib:Qwiic_connector
- added J5: SWD, library:Conn4 1.0mm pitch, symbol mylib:SWDconn4
- added J6: SWD, Connector_PinHeader_2.54mm:PinHeader_1x04_P2.54mm_Vertical_SMD_Pin1Left, symbol mylib:SWDconn4
- added J7: GPIO_header, Connector_PinHeader_2.54mm:PinHeader_1x04_P2.54mm_Vertical_SMD_Pin1Left, symbol Connector:Conn_01x04_Male
- added J8: Debug_header, Connector_PinHeader_2.54mm:PinHeader_1x06_P2.54mm_Vertical_SMD_Pin1Left, symbol Connector:Conn_01x06_Male
- added R7, R8: 1K, Resistor_SMD:R_0603_1608Metric_Pad1.05x0.95mm_HandSolder, symbol Device:R
- added R9: 220R, Resistor_SMD:R_0603_1608Metric_Pad1.05x0.95mm_HandSolder, symbol Device:R
- added TP10: TP_GPIO3, TestPoint:TestPoint_Pad_D1.0mm, symbol Connector:TestPoint
- R1, R2, R3, R4, R5, R6: footprint Resistor_SMD:R_0603_1608Metric -> Resistor_SMD:R_0603_1608Metric_Pad1.05x0.95mm_HandSolder
- TP3: value UART_TX -> TP_UART_TX
- TP4: value VDD -> TP_VCC
- TP5: value GND -> TP_GND
- TP6: value UART_TX -> TP_UART_RX
- TP7: value UART_TX -> TP_GPIO0
- TP8: value UART_TX -> TP_GPIO1
- TP9: value UART_TX -> TP_GPIO2
Connections:
- net +3V3: now also J3.2 (VCC), J5.1 (VCC), J6.1 (VCC), J8.1 (Pin_1), R9.1
- net GND: now also D1.1 (K), D2.1 (K), D3.1 (K), J3.1 (GND), J5.4 (GND), J6.4 (GND), J8.4 (Pin_4)
- net GPIO0: now also J7.1 (Pin_1)
- net GPIO1: now also J7.2 (Pin_2)
- net GPIO2: now also J7.3 (Pin_3), R7.1
- net SCL: now also J3.4 (SCL)
- net SDA: now also J3.3 (SDA)
- net SWCLK: now also J5.3 (SWC), J6.3 (SWC), J8.5 (Pin_5)
- net SWDIO: now also J5.2 (SWD), J6.2 (SWD), J8.6 (Pin_6)
- net UART_RX: now also J8.2 (Pin_2)
- net UART_TX: now also J8.3 (Pin_3)
- net VDDCORE: now reaches C3.1, U2.29 (VDDCORE)
- net GPIO3: now reaches U2.27 (PA28)
- net GPIO3: now also J7.4 (Pin_4), R8.1, TP10.1
- new net: D1.2 (A), R7.2
- new net: D2.2 (A), R8.2
- new net: D3.2 (A), R9.2
- no-connect marks 9 -> 8
Other:
- note added: "CONNECTORS"
- note added: "LEDS"
- note added: "PIN HEADERS"
- note added: "POWER SUPPLY"
- moved on the sheet: C1, C2, C3, J1, J2, J4, Q1, R1, R2, R3, R4, R5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
